Commit message: fixed missing tag liebe 5

File: description/robot.urdf.xacro (robot description, xacro)
@@ -2,5 +2,5 @@
 <robot xmlns:xacro="http://ros.org/wiki/xacro" name="my_robot">
   <!-- Xacro Properties -->
-  <xacro:property name="mesh_file" value="package://ROS2LAUNCH/description/meshes/ATV.DAE">
+  <xacro:property name="mesh_file" value="package://ROS2LAUNCH/description/meshes/ATV.DAE"/>
   <xacro:property name="mesh_scale" value="1 1 1"/>
   <xacro:property name="collision_box_size" value="0.4 0.3 0.2"/>

Commit message: fixed urdf dae path

File: description/robot.urdf.xacro (robot description, xacro)
@@ -2,5 +2,5 @@
 <robot xmlns:xacro="http://ros.org/wiki/xacro" name="my_robot">
   <!-- Xacro Properties -->
-  <xacro:property name="mesh_file" value="package://ROS2LAUNCH/description/meshes/ATV.DAE"/>
+  <xacro:property name="mesh_file" value="package://my_bot/description/meshes/ATV.DAE"/>
   <xacro:property name="mesh_scale" value="1 1 1"/>
   <xacro:property name="collision_box_size" value="0.4 0.3 0.2"/>

Commit message: ACTUALLY fixed urdf pathing

File: description/robot.urdf.xacro (robot description, xacro)
@@ -2,5 +2,5 @@
 <robot xmlns:xacro="http://ros.org/wiki/xacro" name="my_robot">
   <!-- Xacro Properties -->
-  <xacro:property name="mesh_file" value="package://my_bot/description/meshes/ATV.DAE"/>
+  <xacro:property name="mesh_file" value="package://ros2launch/description/meshes/ATV.DAE"/>
   <xacro:property name="mesh_scale" value="1 1 1"/>
   <xacro:property name="collision_box_size" value="0.4 0.3 0.2"/>

Commit message: changed path again

File: description/robot.urdf.xacro (robot description, xacro)
@@ -2,5 +2,5 @@
 <robot xmlns:xacro="http://ros.org/wiki/xacro" name="my_robot">
   <!-- Xacro Properties -->
-  <xacro:property name="mesh_file" value="package://ros2launch/description/meshes/ATV.DAE"/>
+  <xacro:property name="mesh_file" value="/home/kenjif/ros2_ws2/install/my_bot/share/my_bot/description/meshes/ATV.DAE"/>
   <xacro:property name="mesh_scale" value="1 1 1"/>
   <xacro:property name="collision_box_size" value="0.4 0.3 0.2"/>

Commit message: path....

File: description/robot.urdf.xacro (robot description, xacro)
@@ -2,5 +2,5 @@
 <robot xmlns:xacro="http://ros.org/wiki/xacro" name="my_robot">
   <!-- Xacro Properties -->
-  <xacro:property name="mesh_file" value="/home/kenjif/ros2_ws2/install/my_bot/share/my_bot/description/meshes/ATV.DAE"/>
+  <xacro:property name="mesh_file" value="/home/kenjif/ros2_ws2/src/ros2launch/description/meshes/ATV.DAE"/>
   <xacro:property name="mesh_scale" value="1 1 1"/>
   <xacro:property name="collision_box_size" value="0.4 0.3 0.2"/>

Commit message: ughhhhh

File: description/robot.urdf.xacro (robot description, xacro)
@@ -2,5 +2,5 @@
 <robot xmlns:xacro="http://ros.org/wiki/xacro" name="my_robot">
   <!-- Xacro Properties -->
-  <xacro:property name="mesh_file" value="/home/kenjif/ros2_ws2/src/ros2launch/description/meshes/ATV.DAE"/>
+  <xacro:property name="mesh_file" value="/home/kenjif/ros2_ws2/src/ros2launch/description/meshes/ATV.dae"/>
   <xacro:property name="mesh_scale" value="1 1 1"/>
   <xacro:property name="collision_box_size" value="0.4 0.3 0.2"/>

Commit message: 1326yt54

File: description/robot.urdf.xacro (robot description, xacro)
@@ -2,5 +2,5 @@
 <robot xmlns:xacro="http://ros.org/wiki/xacro" name="my_robot">
   <!-- Xacro Properties -->
-  <xacro:property name="mesh_file" value="/home/kenjif/ros2_ws2/src/ros2launch/description/meshes/ATV.dae"/>
+  <mesh filename="package://my_bot/description/meshes/ATV.dae"/>
   <xacro:property name="mesh_scale" value="1 1 1"/>
   <xacro:property name="collision_box_size" value="0.4 0.3 0.2"/>

Commit message: 357567

File: description/robot.urdf.xacro (robot description, xacro)
@@ -2,5 +2,5 @@
 <robot xmlns:xacro="http://ros.org/wiki/xacro" name="my_robot">
   <!-- Xacro Properties -->
-  <mesh filename="package://my_bot/description/meshes/ATV.dae"/>
+  <xacro:property name="mesh_file" value="package://my_bot/description/meshes/ATV.dae"/>
   <xacro:property name="mesh_scale" value="1 1 1"/>
   <xacro:property name="collision_box_size" value="0.4 0.3 0.2"/>

Commit message: added world/joint link

File: description/robot.urdf.xacro (robot description, xacro)
@@ -30,3 +30,11 @@
     </inertial>
   </link>
+  <!-- Add a world link to anchor the robot -->
+  <link name="world"/>
+  <!-- Fixed joint from world to base_link -->
+  <joint name="base_fixed_joint" type="fixed">
+    <parent link="world"/>
+    <child link="base_link"/>
+    <origin xyz="0 0 0" rpy="0 0 0"/>
+  </joint>
 </robot>

Commit message: added camera

File: description/robot.urdf.xacro (robot description, xacro)
@@ -30,4 +30,21 @@
     </inertial>
   </link>
+    <!-- Camera Link -->
+<link name="camera_link">
+  <visual>
+    <geometry>
+      <box size="0.04 0.04 0.03"/>
+    </geometry>
+    <origin xyz="0 0 0" rpy="0 0 0"/>
+    <material name="green"><color rgba="0 1 0 1"/></material>
+  </visual>
+</link>
+<!-- Joint to attach Camera to base_link -->
+<joint name="camera_joint" type="fixed">
+  <parent link="base_link"/>
+  <child link="camera_link"/>
+  <origin xyz="0.1 0 0.2" rpy="0 0 0"/>
+</joint>
+  <!--REMOVE WHEN USING SLAM/NAVIGATION-->
   <!-- Add a world link to anchor the robot -->
   <link name="world"/>

Commit message: update camlink for vm

File: description/robot.urdf.xacro (robot description, xacro)
@@ -9,4 +9,5 @@
   <xacro:property name="iyy" value="0.2"/>
   <xacro:property name="izz" value="0.2"/>
+  <!--THIS IS NOT IN WSL YET DO NOT GIT PULL FROM TTHERE-->
   <!-- Robot Base Link -->
   <link name="base_link">
@@ -31,19 +32,48 @@
   </link>
     <!-- Camera Link -->
-<link name="camera_link">
-  <visual>
-    <geometry>
-      <box size="0.04 0.04 0.03"/>
-    </geometry>
-    <origin xyz="0 0 0" rpy="0 0 0"/>
-    <material name="green"><color rgba="0 1 0 1"/></material>
-  </visual>
-</link>
-<!-- Joint to attach Camera to base_link -->
-<joint name="camera_joint" type="fixed">
-  <parent link="base_link"/>
-  <child link="camera_link"/>
-  <origin xyz="0.1 0 0.2" rpy="0 0 0"/>
-</joint>
+ <joint name="camera_joint" type="fixed">
+        <parent link="base_link"/>
+        <child link="camera_link"/>
+        <origin xyz="0.305 0 0.08" rpy="0 0 0"/>
+    </joint>
+    <link name="camera_link">
+        <visual>
+            <geometry>
+                <box size="0.010 0.03 0.03"/>
+            </geometry>
+            <material name="red"/>
+        </visual>
+    </link>
+    <joint name="camera_optical_joint" type="fixed">
+        <parent link="camera_link"/>
+        <child link="camera_link_optical"/>
+        <origin xyz="0 0 0" rpy="${-pi/2} 0 ${-pi/2}"/>
+    </joint>
+    <link name="camera_link_optical"></link>
+    <gazebo reference="camera_link">
+        <material>Gazebo/Red</material>
+        <sensor name="camera" type="depth">
+            <pose> 0 0 0 0 0 0 </pose>
+            <visualize>true</visualize>
+            <update_rate>10</update_rate>
+            <camera>
+                <horizontal_fov>1.089</horizontal_fov>
+                <image>
+                    <format>B8G8R8</format>
+                    <width>640</width>
+                    <height>480</height>
+                </image>
+                <clip>
+                    <near>0.05</near>
+                    <far>8.0</far>
+                </clip>
+            </camera>
+            <plugin name="camera_controller" filename="libgazebo_ros_camera.so">
+                <frame_name>camera_link_optical</frame_name>
+                <min_depth>0.1</min_depth>
+                <max_depth>100.0</max_depth>
+            </plugin>
+        </sensor>
+    </gazebo>
   <!--REMOVE WHEN USING SLAM/NAVIGATION-->
   <!-- Add a world link to anchor the robot -->

Commit message: removed cam link

File: description/robot.urdf.xacro (robot description, xacro)
@@ -9,71 +9,4 @@
   <xacro:property name="iyy" value="0.2"/>
   <xacro:property name="izz" value="0.2"/>
-  <!--THIS IS NOT IN WSL YET DO NOT GIT PULL FROM TTHERE-->
-  <!-- Robot Base Link -->
-  <link name="base_link">
-    <visual>
-      <geometry>
-        <mesh filename="${mesh_file}" scale="${mesh_scale}"/>
-      </geometry>
-    </visual>
-    <collision>
-      <geometry>
-        <box size="${collision_box_size}"/>
-      </geometry>
-    </collision>
-    <inertial>
-      <mass value="${mass_kg}"/>
-      <origin xyz="0 0 0" rpy="0 0 0"/>
-      <inertia
-        ixx="${ixx}" ixy="0.0" ixz="0.0"
-        iyy="${iyy}" iyz="0.0"
-        izz="${izz}"/>
-    </inertial>
-  </link>
-    <!-- Camera Link -->
- <joint name="camera_joint" type="fixed">
-        <parent link="base_link"/>
-        <child link="camera_link"/>
-        <origin xyz="0.305 0 0.08" rpy="0 0 0"/>
-    </joint>
-    <link name="camera_link">
-        <visual>
-            <geometry>
-                <box size="0.010 0.03 0.03"/>
-            </geometry>
-            <material name="red"/>
-        </visual>
-    </link>
-    <joint name="camera_optical_joint" type="fixed">
-        <parent link="camera_link"/>
-        <child link="camera_link_optical"/>
-        <origin xyz="0 0 0" rpy="${-pi/2} 0 ${-pi/2}"/>
-    </joint>
-    <link name="camera_link_optical"></link>
-    <gazebo reference="camera_link">
-        <material>Gazebo/Red</material>
-        <sensor name="camera" type="depth">
-            <pose> 0 0 0 0 0 0 </pose>
-            <visualize>true</visualize>
-            <update_rate>10</update_rate>
-            <camera>
-                <horizontal_fov>1.089</horizontal_fov>
-                <image>
-                    <format>B8G8R8</format>
-                    <width>640</width>
-                    <height>480</height>
-                </image>
-                <clip>
-                    <near>0.05</near>
-                    <far>8.0</far>
-                </clip>
-            </camera>
-            <plugin name="camera_controller" filename="libgazebo_ros_camera.so">
-                <frame_name>camera_link_optical</frame_name>
-                <min_depth>0.1</min_depth>
-                <max_depth>100.0</max_depth>
-            </plugin>
-        </sensor>
-    </gazebo>
   <!--REMOVE WHEN USING SLAM/NAVIGATION-->
   <!-- Add a world link to anchor the robot -->

Commit message: fixed base link

File: description/robot.urdf.xacro (robot description, xacro)
@@ -9,4 +9,24 @@
   <xacro:property name="iyy" value="0.2"/>
   <xacro:property name="izz" value="0.2"/>
+  <link name="base_link">
+    <visual>
+      <geometry>
+        <mesh filename="${mesh_file}" scale="${mesh_scale}"/>
+      </geometry>
+    </visual>
+    <collision>
+      <geometry>
+        <box size="${collision_box_size}"/>
+      </geometry>
+    </collision>
+    <inertial>
+      <mass value="${mass_kg}"/>
+      <origin xyz="0 0 0" rpy="0 0 0"/>
+      <inertia
+        ixx="${ixx}" ixy="0.0" ixz="0.0"
+        iyy="${iyy}" iyz="0.0"
+        izz="${izz}"/>
+    </inertial>
+  </link>
   <!--REMOVE WHEN USING SLAM/NAVIGATION-->
   <!-- Add a world link to anchor the robot -->

Commit message: added wheels/camera

File: description/robot.urdf.xacro (robot description, xacro)
@@ -29,4 +29,49 @@
     </inertial>
   </link>
+    <!-- Four Wheels -->
+  <xacro:macro name="wheel" params="name x y">
+    <link name="${name}">
+      <visual>
+        <geometry>
+          <cylinder radius="${wheel_radius}" length="${wheel_width}"/>
+        </geometry>
+        <origin xyz="0 0 0" rpy="0 1.5708 0"/>
+        <material name="black">
+          <color rgba="0.1 0.1 0.1 1"/>
+        </material>
+      </visual>
+    </link>
+    <joint name="${name}_joint" type="fixed">
+      <parent link="base_link"/>
+      <child link="${name}"/>
+      <origin xyz="${x} ${y} -${wheel_radius}" rpy="0 0 0"/>
+    </joint>
+  </xacro:macro>
+  <xacro:wheel name="front_left_wheel"  x="0.2"  y="0.15"/>
+  <xacro:wheel name="front_right_wheel" x="0.2"  y="-0.15"/>
+  <xacro:wheel name="rear_left_wheel"   x="-0.2" y="0.15"/>
+  <xacro:wheel name="rear_right_wheel"  x="-0.2" y="-0.15"/>
+  <!-- Camera -->
+  <link name="camera_link">
+    <visual>
+      <geometry>
+        <box size="0.05 0.05 0.05"/>
+      </geometry>
+      <material name="blue">
+        <color rgba="0.1 0.1 1 1"/>
+      </material>
+    </visual>
+  </link>
+  <joint name="camera_joint" type="fixed">
+    <parent link="base_link"/>
+    <child link="camera_link"/>
+    <origin xyz="0.3 0 0.1" rpy="0 0 0"/>
+  </joint>
+  <link name="camera_link_optical"/>
+  <joint name="camera_optical_joint" type="fixed">
+    <parent link="camera_link"/>
+    <child link="camera_link_optical"/>
+    <origin xyz="0 0 0" rpy="${-pi/2} 0 ${-pi/2}"/>
+  </joint>
   <!--REMOVE WHEN USING SLAM/NAVIGATION-->
   <!-- Add a world link to anchor the robot -->

Commit message: added wheel properties

File: description/robot.urdf.xacro (robot description, xacro)
@@ -9,4 +9,6 @@
   <xacro:property name="iyy" value="0.2"/>
   <xacro:property name="izz" value="0.2"/>
+  <xacro:property name="wheel_radius" value="0.1"/>
+  <xacro:property name="wheel_width" value="0.05"/>
   <link name="base_link">
     <visual>

Commit message: removed wheels for now

File: description/robot.urdf.xacro (robot description, xacro)
@@ -31,27 +31,4 @@
     </inertial>
   </link>
-    <!-- Four Wheels -->
-  <xacro:macro name="wheel" params="name x y">
-    <link name="${name}">
-      <visual>
-        <geometry>
-          <cylinder radius="${wheel_radius}" length="${wheel_width}"/>
-        </geometry>
-        <origin xyz="0 0 0" rpy="0 1.5708 0"/>
-        <material name="black">
-          <color rgba="0.1 0.1 0.1 1"/>
-        </material>
-      </visual>
-    </link>
-    <joint name="${name}_joint" type="fixed">
-      <parent link="base_link"/>
-      <child link="${name}"/>
-      <origin xyz="${x} ${y} -${wheel_radius}" rpy="0 0 0"/>
-    </joint>
-  </xacro:macro>
-  <xacro:wheel name="front_left_wheel"  x="0.2"  y="0.15"/>
-  <xacro:wheel name="front_right_wheel" x="0.2"  y="-0.15"/>
-  <xacro:wheel name="rear_left_wheel"   x="-0.2" y="0.15"/>
-  <xacro:wheel name="rear_right_wheel"  x="-0.2" y="-0.15"/>
   <!-- Camera -->
   <link name="camera_link">

Commit message: added depth cam

File: description/robot.urdf.xacro (robot description, xacro)
@@ -53,4 +53,29 @@
     <origin xyz="0 0 0" rpy="${-pi/2} 0 ${-pi/2}"/>
   </joint>
+  <gazebo reference="camera_link">
+        <material>Gazebo/Red</material>
+        <sensor name="camera" type="depth">
+            <pose> 0 0 0 0 0 0 </pose>
+            <visualize>true</visualize>
+            <update_rate>10</update_rate>
+            <camera>
+                <horizontal_fov>1.089</horizontal_fov>
+                <image>
+                    <format>B8G8R8</format>
+                    <width>640</width>
+                    <height>480</height>
+                </image>
+                <clip>
+                    <near>0.05</near>
+                    <far>8.0</far>
+                </clip>
+            </camera>
+            <plugin name="camera_controller" filename="libgazebo_ros_camera.so">
+                <frame_name>camera_link_optical</frame_name>
+                <min_depth>0.1</min_depth>
+                <max_depth>100.0</max_depth>
+            </plugin>
+        </sensor>
+    </gazebo>
   <!--REMOVE WHEN USING SLAM/NAVIGATION-->
   <!-- Add a world link to anchor the robot -->

Commit message: updated camera

File: description/robot.urdf.xacro (robot description, xacro)
@@ -32,50 +32,53 @@
   </link>
   <!-- Camera -->
-  <link name="camera_link">
-    <visual>
-      <geometry>
-        <box size="0.05 0.05 0.05"/>
-      </geometry>
-      <material name="blue">
-        <color rgba="0.1 0.1 1 1"/>
-      </material>
-    </visual>
-  </link>
-  <joint name="camera_joint" type="fixed">
-    <parent link="base_link"/>
-    <child link="camera_link"/>
-    <origin xyz="0.3 0 0.1" rpy="0 0 0"/>
-  </joint>
-  <link name="camera_link_optical"/>
-  <joint name="camera_optical_joint" type="fixed">
-    <parent link="camera_link"/>
-    <child link="camera_link_optical"/>
-    <origin xyz="0 0 0" rpy="${-pi/2} 0 ${-pi/2}"/>
-  </joint>
-  <gazebo reference="camera_link">
-        <material>Gazebo/Red</material>
-        <sensor name="camera" type="depth">
-            <pose> 0 0 0 0 0 0 </pose>
-            <visualize>true</visualize>
-            <update_rate>10</update_rate>
-            <camera>
-                <horizontal_fov>1.089</horizontal_fov>
-                <image>
-                    <format>B8G8R8</format>
-                    <width>640</width>
-                    <height>480</height>
-                </image>
-                <clip>
-                    <near>0.05</near>
-                    <far>8.0</far>
-                </clip>
-            </camera>
-            <plugin name="camera_controller" filename="libgazebo_ros_camera.so">
-                <frame_name>camera_link_optical</frame_name>
-                <min_depth>0.1</min_depth>
-                <max_depth>100.0</max_depth>
-            </plugin>
-        </sensor>
-    </gazebo>
+  <!-- Camera Link -->
+<link name="camera_link">
+  <visual>
+    <geometry>
+      <box size="0.05 0.05 0.05"/>
+    </geometry>
+    <material name="blue">
+      <color rgba="0.1 0.1 1 1"/>
+    </material>
+  </visual>
+</link>
+<!-- Camera Mount Joint -->
+<joint name="camera_joint" type="fixed">
+  <parent link="base_link"/>
+  <child link="camera_link"/>
+  <origin xyz="0.3 0 0.1" rpy="0 0 0"/>
+</joint>
+<!-- Optical Link (standard for camera frames) -->
+<link name="camera_link_optical"/>
+<joint name="camera_optical_joint" type="fixed">
+  <parent link="camera_link"/>
+  <child link="camera_link_optical"/>
+  <origin xyz="0 0 0" rpy="${-pi/2} 0 ${-pi/2}"/>
+</joint>
+<!-- Gazebo Harmonic Camera Sensor -->
+<gazebo reference="camera_link">
+  <sensor name="depth_camera" type="camera">
+    <camera>
+      <horizontal_fov>1.089</horizontal_fov>
+      <image>
+        <width>640</width>
+        <height>480</height>
+        <format>R8G8B8</format>
+      </image>
+      <clip>
+        <near>0.1</near>
+        <far>10.0</far>
+      </clip>
+    </camera>
+    <plugin name="camera_controller" filename="libgz_ros_camera_system.so">
+      <ros>
+        <namespace>/camera</namespace>
+        <remapping>image_raw:=image_raw</remapping>
+      </ros>
+      <camera_name>camera</camera_name>
+      <frame_name>camera_link_optical</frame_name>
+    </plugin>
+  </sensor>
+</gazebo>
   <!--REMOVE WHEN USING SLAM/NAVIGATION-->
   <!-- Add a world link to anchor the robot -->

Commit message: updated camera again

File: description/robot.urdf.xacro (robot description, xacro)
@@ -33,32 +33,11 @@
   <!-- Camera -->
   <!-- Camera Link -->
-<link name="camera_link">
-  <visual>
-    <geometry>
-      <box size="0.05 0.05 0.05"/>
-    </geometry>
-    <material name="blue">
-      <color rgba="0.1 0.1 1 1"/>
-    </material>
-  </visual>
-</link>
-<!-- Camera Mount Joint -->
-<joint name="camera_joint" type="fixed">
-  <parent link="base_link"/>
-  <child link="camera_link"/>
-  <origin xyz="0.3 0 0.1" rpy="0 0 0"/>
-</joint>
-<!-- Optical Link (standard for camera frames) -->
-<link name="camera_link_optical"/>
-<joint name="camera_optical_joint" type="fixed">
-  <parent link="camera_link"/>
-  <child link="camera_link_optical"/>
-  <origin xyz="0 0 0" rpy="${-pi/2} 0 ${-pi/2}"/>
-</joint>
-<!-- Gazebo Harmonic Camera Sensor -->
-<gazebo reference="camera_link">
-  <sensor name="depth_camera" type="camera">
+ <gazebo reference="camera_link">
+  <sensor name="camera" type="depth">
+    <pose>0 0 0 0 0 0</pose>
+    <visualize>true</visualize>
+    <update_rate>30.0</update_rate>
     <camera>
-      <horizontal_fov>1.089</horizontal_fov>
+      <horizontal_fov>1.047</horizontal_fov>
       <image>
         <width>640</width>
@@ -71,14 +50,10 @@
       </clip>
     </camera>
-    <plugin name="camera_controller" filename="libgz_ros_camera_system.so">
-      <ros>
-        <namespace>/camera</namespace>
-        <remapping>image_raw:=image_raw</remapping>
-      </ros>
+    <plugin name="camera_controller" filename="libgazebo_ros_camera.so">
       <camera_name>camera</camera_name>
       <frame_name>camera_link_optical</frame_name>
     </plugin>
   </sensor>
-</gazebo>
+ </gazebo>
   <!--REMOVE WHEN USING SLAM/NAVIGATION-->
   <!-- Add a world link to anchor the robot -->

Commit message: updated cam/rsp launch

File: description/robot.urdf.xacro (robot description, xacro)
@@ -33,7 +33,29 @@
   <!-- Camera -->
   <!-- Camera Link -->
- <gazebo reference="camera_link">
-  <sensor name="camera" type="camera">
-    <update_rate>30.0</update_rate>
+ <!-- Attach camera to base_link -->
+<joint name="camera_joint" type="fixed">
+  <parent link="base_link"/>
+  <child link="camera_link"/>
+  <origin xyz="0.3 0 0.1" rpy="0 0 0"/>
+</joint>
+<link name="camera_link">
+  <visual>
+    <geometry>
+      <box size="0.05 0.05 0.05"/>
+    </geometry>
+    <material name="grey"/>
+  </visual>
+</link>
+<!-- Optional optical frame if needed -->
+<joint name="camera_optical_joint" type="fixed">
+  <parent link="camera_link"/>
+  <child link="camera_link_optical"/>
+  <origin xyz="0 0 0" rpy="${-pi/2} 0 ${-pi/2}"/>
+</joint>
+<link name="camera_link_optical" />
+<!-- Gazebo Harmonic camera sensor -->
+<gazebo reference="camera_link">
+  <sensor name="camera_sensor" type="camera">
+    <pose>0 0 0 0 0 0</pose>
     <camera>
       <horizontal_fov>1.047</horizontal_fov>
@@ -48,5 +70,8 @@
       </clip>
     </camera>
-    <plugin name="camera_controller" filename="libgazebo_ros_camera.so"/>
+    <plugin
+      name="camera_controller"
+      filename="libgz_ros_camera_system.so">
+    </plugin>
   </sensor>
 </gazebo>
