Commit message: seperated wheel/chassis

File: description/robot.urdf.xacro (robot description, xacro)
@@ -2,5 +2,5 @@
 <robot xmlns:xacro="http://ros.org/wiki/xacro" name="my_robot">
   <!-- Xacro Properties -->
-  <xacro:property name="mesh_file" value="package://my_bot/description/meshes/ATV.dae"/>
+  <xacro:property name="body_mesh_file" value="package://my_bot/description/meshes/ATV_Chassis.dae"/>
   <xacro:property name="mesh_scale" value="1 1 1"/>
   <xacro:property name="collision_box_size" value="0.4 0.3 0.2"/>
@@ -11,8 +11,12 @@
   <xacro:property name="wheel_radius" value="0.1"/>
   <xacro:property name="wheel_width" value="0.05"/>
+    <!-- Load wheel macro -->
+  <xacro:include filename="wheel_macro.xacro"/>
+  <!-- Define mesh path once -->
+  <xacro:property name="wheel_mesh" value="package://my_bot/description/meshes/wheel.dae"/>
   <link name="base_link">
     <visual>
       <geometry>
-        <mesh filename="${mesh_file}" scale="${mesh_scale}"/>
+        <mesh filename="${body_mesh_file}" scale="${mesh_scale}"/>
       </geometry>
     </visual>
@@ -31,49 +35,9 @@
     </inertial>
   </link>
-  <!-- Camera -->
-  <!-- Camera Link -->
- <!-- Attach camera to base_link -->
-<joint name="camera_joint" type="fixed">
-  <parent link="base_link"/>
-  <child link="camera_link"/>
-  <origin xyz="0.3 0 0.1" rpy="0 0 0"/>
-</joint>
-<link name="camera_link">
-  <visual>
-    <geometry>
-      <box size="0.05 0.05 0.05"/>
-    </geometry>
-    <material name="grey"/>
-  </visual>
-</link>
-<!-- Optional optical frame if needed -->
-<joint name="camera_optical_joint" type="fixed">
-  <parent link="camera_link"/>
-  <child link="camera_link_optical"/>
-  <origin xyz="0 0 0" rpy="${-pi/2} 0 ${-pi/2}"/>
-</joint>
-<link name="camera_link_optical" />
-<!-- Gazebo Harmonic camera sensor -->
-<gazebo reference="camera_link">
-  <sensor name="camera_sensor" type="camera">
-    <pose>0 0 0 0 0 0</pose>
-    <camera>
-      <horizontal_fov>1.047</horizontal_fov>
-      <image>
-        <width>640</width>
-        <height>480</height>
-        <format>R8G8B8</format>
-      </image>
-      <clip>
-        <near>0.1</near>
-        <far>10.0</far>
-      </clip>
-    </camera>
-    <plugin
-      name="camera_controller"
-      filename="libgz_ros_camera_system.so">
-    </plugin>
-  </sensor>
-</gazebo>
+    <!-- Add 4 wheels -->
+  <xacro:add_wheel wheel_name="front_left_wheel"  xyz="0.3  0.2  0.05" rpy="0 0 0" mesh="${wheel_mesh}"/>
+  <xacro:add_wheel wheel_name="front_right_wheel" xyz="0.3 -0.2  0.05" rpy="0 0 0" mesh="${wheel_mesh}"/>
+  <xacro:add_wheel wheel_name="rear_left_wheel"   xyz="-0.3  0.2  0.05" rpy="0 0 0" mesh="${wheel_mesh}"/>
+  <xacro:add_wheel wheel_name="rear_right_wheel"  xyz="-0.3 -0.2  0.05" rpy="0 0 0" mesh="${wheel_mesh}"/>
   <!--REMOVE WHEN USING SLAM/NAVIGATION-->
   <!-- Add a world link to anchor the robot -->

Commit message: fixed all wheel pathing names i think

File: description/robot.urdf.xacro (robot description, xacro)
@@ -12,7 +12,7 @@
   <xacro:property name="wheel_width" value="0.05"/>
     <!-- Load wheel macro -->
-  <xacro:include filename="$(find my_bot)/description/wheel_macro.xacro" />
+  <xacro:include filename="wheel_macro.xacro" />
   <!-- Define mesh path once -->
-  <xacro:property name="wheel_mesh" value="package://my_bot/description/meshes/wheel.dae"/>
+  <xacro:property name="wheel_mesh" value="package://my_bot/description/meshes/Wheel.dae"/>
   <link name="base_link">
     <visual>

Commit message: added new gazebo files

File: description/robot.urdf.xacro (robot description, xacro)
@@ -1,54 +1,93 @@
 <?xml version="1.0"?>
-<robot xmlns:xacro="http://ros.org/wiki/xacro" name="my_robot">
-  <xacro:arg name="use_ros2_control" default="true"/>
-  <xacro:arg name="sim_mode" default="false"/>
-  <!-- Xacro Properties -->
+<robot name="atv_bot" xmlns:xacro="http://www.ros.org/wiki/xacro">
+  <!-- Xacro Includes -->
+  <xacro:include filename="robot.gazebo"/>
+  <xacro:include filename="wheel_macro.xacro"/>
+  <!-- Mesh properties -->
   <xacro:property name="body_mesh_file" value="package://my_bot/description/meshes/ATV_Chassis.dae"/>
+  <xacro:property name="wheel_mesh" value="package://my_bot/description/meshes/Wheel.dae"/>
   <xacro:property name="mesh_scale" value="1 1 1"/>
-  <xacro:property name="collision_box_size" value="0.4 0.3 0.2"/>
-  <xacro:property name="mass_kg" value="5.0"/>
-  <xacro:property name="ixx" value="0.2"/>
-  <xacro:property name="iyy" value="0.2"/>
-  <xacro:property name="izz" value="0.2"/>
-  <xacro:property name="wheel_radius" value="0.1"/>
-  <xacro:property name="wheel_width" value="0.05"/>
-  <xacro:include filename="camera.xacro" />
-    <!-- Load wheel macro -->
-  <xacro:include filename="wheel_macro.xacro" />
-  <!-- Define mesh path once -->
-  <xacro:property name="wheel_mesh" value="package://my_bot/description/meshes/Wheel.dae"/>
+  <!-- Frame root for SLAM/navigation -->
+  <link name="base_footprint"/>
+  <joint name="base_footprint_joint" type="fixed">
+    <origin xyz="0 0 0" rpy="0 0 0"/>
+    <parent link="base_footprint"/>
+    <child link="base_link"/>
+  </joint>
+  <!-- Base Link using ATV chassis -->
   <link name="base_link">
+    <inertial>
+      <mass value="15.0"/>
+      <origin xyz="0 0 0" rpy="0 0 0"/>
+      <inertia ixx="0.0625" ixy="0" ixz="0" iyy="0.2125" iyz="0" izz="0.25"/>
+    </inertial>
+    <collision>
+      <origin xyz="0 0 0" rpy="0 0 0"/>
+      <geometry>
+        <box size="0.4 0.3 0.2"/>
+      </geometry>
+    </collision>
     <visual>
+      <origin xyz="0 0 0" rpy="0 0 0"/>
       <geometry>
         <mesh filename="${body_mesh_file}" scale="${mesh_scale}"/>
       </geometry>
     </visual>
-    <collision>
-      <geometry>
-        <box size="${collision_box_size}"/>
-      </geometry>
-    </collision>
-    <inertial>
-      <mass value="${mass_kg}"/>
-      <origin xyz="0 0 0" rpy="0 0 0"/>
-      <inertia
-        ixx="${ixx}" ixy="0.0" ixz="0.0"
-        iyy="${iyy}" iyz="0.0"
-        izz="${izz}"/>
-    </inertial>
   </link>
-    <!-- Add 4 wheels -->
+  <!-- Wheels using macro (you must define the macro in wheel_macro.xacro) -->
   <xacro:add_wheel wheel_name="front_left_wheel"  xyz="0.3  0.2  0.05" rpy="0 0 0" mesh="${wheel_mesh}"/>
   <xacro:add_wheel wheel_name="front_right_wheel" xyz="0.3 -0.2  0.05" rpy="0 0 0" mesh="${wheel_mesh}"/>
   <xacro:add_wheel wheel_name="rear_left_wheel"   xyz="-0.3  0.2  0.05" rpy="0 0 0" mesh="${wheel_mesh}"/>
   <xacro:add_wheel wheel_name="rear_right_wheel"  xyz="-0.3 -0.2  0.05" rpy="0 0 0" mesh="${wheel_mesh}"/>
-  <!--REMOVE WHEN USING SLAM/NAVIGATION-->
-  <!-- Add a world link to anchor the robot -->
-  <link name="world"/>
-  <!-- Fixed joint from world to base_link -->
-  <joint name="base_fixed_joint" type="fixed">
-    <parent link="world"/>
-    <child link="base_link"/>
+  <!-- Camera -->
+  <joint type="fixed" name="camera_joint">
+    <origin xyz="0.225 0 0.075" rpy="0 0 0"/>
+    <parent link="base_link"/>
+    <child link="camera_link"/>
+  </joint>
+  <link name="camera_link">
+    <inertial>
+      <mass value="0.1"/>
+      <origin xyz="0 0 0" rpy="0 0 0"/>
+      <inertia ixx="1e-6" ixy="0" ixz="0" iyy="1e-6" iyz="0" izz="1e-6"/>
+    </inertial>
+    <collision>
+      <geometry><box size="0.03 0.03 0.03"/></geometry>
+    </collision>
+    <visual>
+      <geometry><box size="0.03 0.03 0.03"/></geometry>
+    </visual>
+  </link>
+  <joint type="fixed" name="camera_optical_joint">
+    <origin xyz="0 0 0" rpy="-1.5707 0 -1.5707"/>
+    <parent link="camera_link"/>
+    <child link="camera_link_optical"/>
+  </joint>
+  <link name="camera_link_optical"/>
+  <!-- IMU -->
+  <joint name="imu_joint" type="fixed">
     <origin xyz="0 0 0" rpy="0 0 0"/>
+    <parent link="base_link"/>
+    <child link="imu_link"/>
   </joint>
+  <link name="imu_link"/>
+  <!-- Lidar -->
+  <joint type="fixed" name="scan_joint">
+    <origin xyz="0.0 0 0.15" rpy="0 0 0"/>
+    <parent link="base_link"/>
+    <child link="scan_link"/>
+  </joint>
+  <link name="scan_link">
+    <inertial>
+      <mass value="1e-5"/>
+      <origin xyz="0 0 0" rpy="0 0 0"/>
+      <inertia ixx="1e-6" ixy="0" ixz="0" iyy="1e-6" iyz="0" izz="1e-6"/>
+    </inertial>
+    <collision>
+      <geometry><box size="0.1 0.1 0.1"/></geometry>
+    </collision>
+    <visual>
+      <geometry><mesh filename="package://bme_ros2_navigation/meshes/lidar.dae"/></geometry>
+    </visual>
+  </link>
 </robot>

Commit message: fixed lidar path in urdf/got rid of worlds uri

File: description/robot.urdf.xacro (robot description, xacro)
@@ -88,5 +88,5 @@
     </collision>
     <visual>
-      <geometry><mesh filename="package://bme_ros2_navigation/meshes/lidar.dae"/></geometry>
+      <geometry><mesh filename="package://my_bot/description/meshes/lidar.dae"/></geometry>
     </visual>
   </link>
